File: shocker.kicad_sch (KiCad schematic)
At the start: 62 parts, among them J1 Barrel_Jack, Q1 KTC4373Y, Q2 Q_NPN_BEC, Q3 Q_NPN_BEC, T11 TestPoint, T15 TestPoint, T16 SHOCKER_OUTPUT_0, T17 TestPoint, T18 V, T19 G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

Commit message: fixed mistake where i didn't specify transistor part number
Parts:
- Q2, Q3: value Q_NPN_BEC -> SS8050
- gave numbers to parts that had none: 1
Changed lines of the file:
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@@
 			)
 		)
-		(property "Value" "Q_NPN_BEC"
+		(property "Value" "SS8050"
 			(at 353.06 120.6499 0)
 			(effects
@@
 			)
 		)
-		(property "Value" "Q_NPN_BEC"
+		(property "Value" "SS8050"
 			(at 245.11 104.1399 0)
 			(effects
@@
 		(dnp no)
 		(fields_autoplaced yes)
-		(property "Reference" "Q?"
+		(property "Reference" "Q5"
 			(at 69.85 142.2399 0)
 			(effects
@@
 			(project "caixianlin_remote_shocker"
 				(path "/c1360231-0ff3-4c3f-a7b5-1142b0ed19a4/16646a8c-b803-44e2-8c15-74c54d1f7943"
-					(reference "Q?")
+					(reference "Q5")
 					(unit 1)
 				)

Commit message: fix dumb issue where i got the power wires on the main chip backward...
Connections:
- net CHARGE_COMPLETE? is gone; now on net CHARGE_COMPLETE: T8.1
- net +3.3V: now also U3.1; no longer U3.16
- net GND: now also U3.16; no longer U3.1
Changed lines of the file:
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@@
 	(wire
 		(pts
+			(xy 64.77 35.56) (xy 68.58 35.56)
+		)
+		(stroke
+			(width 0)
+			(type default)
+		)
+	)
+	(wire
+		(pts
 			(xy 217.17 161.29) (xy 217.17 163.83)
 		)
@@
 	(wire
 		(pts
+			(xy 83.82 35.56) (xy 87.63 35.56)
+		)
+		(stroke
+			(width 0)
+			(type default)
+		)
+	)
+	(wire
+		(pts
 			(xy 201.93 251.46) (xy 213.36 251.46)
 		)
@@
 	(wire
 		(pts
-			(xy 83.82 35.56) (xy 87.63 35.56)
-		)
-		(stroke
-			(width 0)
-			(type default)
-		)
-	)
-	(wire
-		(pts
 			(xy 67.31 133.35) (xy 74.93 133.35)
 		)
@@
 	(wire
 		(pts
-			(xy 64.77 35.56) (xy 68.58 35.56)
-		)
-		(stroke
-			(width 0)
-			(type default)
-		)
-	)
-	(wire
-		(pts
 			(xy 325.12 207.01) (xy 356.87 207.01)
 		)
@@
 		)
 	)
-	(global_label "CHARGE_COMPLETE?"
+	(global_label "CHARGE_COMPLETE"
 		(shape input)
 		(at 168.91 54.61 180)
@@
 		)
 		(property "Intersheetrefs" "${INTERSHEET_REFS}"
-			(at 146.8749 54.61 0)
+			(at 147.9635 54.61 0)
 			(effects
 				(font
@@
 	(symbol
 		(lib_id "power:+3.3V")
-		(at 87.63 35.56 0)
+		(at 64.77 35.56 0)
 		(mirror y)
 		(unit 1)
@@
 		(fields_autoplaced yes)
 		(property "Reference" "#PWR059"
-			(at 87.63 39.37 0)
+			(at 64.77 39.37 0)
 			(effects
 				(font
@@
 		)
 		(property "Value" "+3.3V"
-			(at 87.63 30.48 0)
+			(at 64.77 30.48 0)
 			(effects
 				(font
@@
 		)
 		(property "Footprint" ""
-			(at 87.63 35.56 0)
+			(at 64.77 35.56 0)
 			(effects
 				(font
@@
 		)
 		(property "Datasheet" ""
-			(at 87.63 35.56 0)
+			(at 64.77 35.56 0)
 			(effects
 				(font
@@
 		)
 		(property "Description" "Power symbol creates a global label with name \"+3.3V\""
-			(at 87.63 35.56 0)
+			(at 64.77 35.56 0)
 			(effects
 				(font
@@
 	(symbol
 		(lib_id "power:GND")
-		(at 64.77 35.56 270)
+		(at 87.63 35.56 90)
+		(mirror x)
 		(unit 1)
 		(exclude_from_sim no)
@@
 		(on_board yes)
 		(dnp no)
-		(fields_autoplaced yes)
 		(property "Reference" "#PWR060"
-			(at 58.42 35.56 0)
+			(at 93.98 35.56 0)
 			(effects
 				(font
@@
 		)
 		(property "Value" "GND"
-			(at 60.96 35.5599 90)
+			(at 91.44 35.5599 90)
 			(effects
 				(font
@@
 		)
 		(property "Footprint" ""
-			(at 64.77 35.56 0)
+			(at 87.63 35.56 0)
 			(effects
 				(font
@@
 		)
 		(property "Datasheet" ""
-			(at 64.77 35.56 0)
+			(at 87.63 35.56 0)
 			(effects
 				(font
@@
 		)
 		(property "Description" "Power symbol creates a global label with name \"GND\" , ground"
-			(at 64.77 35.56 0)
+			(at 87.63 35.56 0)
 			(effects
 				(font

Commit message: fix reference values
Parts:
- gave numbers to parts that had none: 2
Changed lines of the file:
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@@
 		(dnp no)
 		(fields_autoplaced yes)
-		(property "Reference" "M?"
+		(property "Reference" "MOTO1"
 			(at 247.65 88.8999 0)
 			(effects
@@
 			(project ""
 				(path "/c1360231-0ff3-4c3f-a7b5-1142b0ed19a4/16646a8c-b803-44e2-8c15-74c54d1f7943"
-					(reference "M?")
+					(reference "MOTO1")
 					(unit 1)
 				)
@@
 		(dnp no)
 		(fields_autoplaced yes)
-		(property "Reference" "AE?"
+		(property "Reference" "ANT1"
 			(at 307.34 197.4849 0)
 			(effects
@@
 			(project ""
 				(path "/c1360231-0ff3-4c3f-a7b5-1142b0ed19a4/16646a8c-b803-44e2-8c15-74c54d1f7943"
-					(reference "AE?")
-					(unit 1)
-				)
+					(reference "ANT1")
+					(unit 1)
+				)

Commit message: update schematic with new info
Parts:
- R10: value 15 -> 0.51 Ohms
- R2: value ? -> 56 Ohms
Other:
- moved on the sheet: L3, Q1, R2, T16, T4
Changed lines of the file:
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@@
 	(wire
 		(pts
-			(xy 351.79 29.21) (xy 351.79 33.02)
+			(xy 335.28 27.94) (xy 335.28 31.75)
 		)
 		(stroke
@@
 	(wire
 		(pts
-			(xy 361.95 33.02) (xy 374.65 33.02)
+			(xy 345.44 31.75) (xy 358.14 31.75)
 		)
 		(stroke
@@
 	(wire
 		(pts
-			(xy 361.95 43.18) (xy 374.65 43.18)
+			(xy 345.44 41.91) (xy 358.14 41.91)
 		)
 		(stroke
@@
 	(wire
 		(pts
-			(xy 351.79 57.15) (xy 351.79 60.96)
+			(xy 335.28 55.88) (xy 335.28 59.69)
 		)
 		(stroke
@@
 	(wire
 		(pts
-			(xy 328.93 52.07) (xy 332.74 52.07)
+			(xy 312.42 50.8) (xy 316.23 50.8)
 		)
 		(stroke
@@
 	(wire
 		(pts
-			(xy 351.79 43.18) (xy 351.79 46.99)
+			(xy 335.28 41.91) (xy 335.28 45.72)
 		)
 		(stroke
@@
 	(wire
 		(pts
-			(xy 340.36 52.07) (xy 344.17 52.07)
+			(xy 323.85 50.8) (xy 327.66 50.8)
 		)
 		(stroke
@@
 		)
 	)
+	(text_box "primary has a resistance of 2.2 Ohms.\nsecondary has a resistance of 2.865K Ohms."
+		(exclude_from_sim no)
+		(at 350.52 50.165 0)
+		(size 46.355 6.35)
+		(stroke
+			(width 0)
+			(type default)
+		)
+		(fill
+			(type none)
+		)
+		(effects
+			(font
+				(size 1.27 1.27)
+			)
+			(justify left top)
+		)
+	)
 	(text_box "NOTE: THE TRANSFORMER HAS A DUMMY PIN THAT MAKES IT LOOKS LIKE THE PRIMARY IS CENTER TAPPED, BUT IT IS NOT CONNECTED INTERNALLY.\n"
 		(exclude_from_sim no)
-		(at 311.15 18.415 0)
+		(at 294.64 17.145 0)
 		(size 27.94 13.97)
 		(stroke
@@
 	(global_label "SHOCK_SIG"
 		(shape input)
-		(at 328.93 52.07 180)
+		(at 312.42 50.8 180)
 		(fields_autoplaced yes)
 		(effects
@@
 		)
 		(property "Intersheetrefs" "${INTERSHEET_REFS}"
-			(at 315.4824 52.07 0)
+			(at 298.9724 50.8 0)
 			(effects
 				(font
@@
 	(symbol
 		(lib_id "power:GND")
-		(at 351.79 60.96 0)
+		(at 335.28 59.69 0)
 		(unit 1)
 		(exclude_from_sim no)
@@
 		(fields_autoplaced yes)
 		(property "Reference" "#PWR057"
-			(at 351.79 67.31 0)
+			(at 335.28 66.04 0)
 			(effects
 				(font
@@
 		)
 		(property "Value" "GND"
-			(at 351.79 66.04 0)
+			(at 335.28 64.77 0)
 			(effects
 				(font
@@
 		)
 		(property "Footprint" ""
-			(at 351.79 60.96 0)
+			(at 335.28 59.69 0)
 			(effects
 				(font
@@
 		)
 		(property "Datasheet" ""
-			(at 351.79 60.96 0)
+			(at 335.28 59.69 0)
 			(effects
 				(font
@@
 		)
 		(property "Description" "Power symbol creates a global label with name \"GND\" , ground"
-			(at 351.79 60.96 0)
+			(at 335.28 59.69 0)
 			(effects
 				(font
@@
 	(symbol
 		(lib_id "Connector:Conn_01x01_Pin")
-		(at 379.73 43.18 180)
+		(at 363.22 41.91 180)
 		(unit 1)
 		(exclude_from_sim no)
@@
 		(fields_autoplaced yes)
 		(property "Reference" "T16"
-			(at 379.095 38.1 0)
+			(at 362.585 36.83 0)
 			(effects
 				(font
@@
 		)
 		(property "Value" "SHOCKER_OUTPUT_0"
-			(at 379.095 40.64 0)
+			(at 362.585 39.37 0)
 			(effects
 				(font
@@
 		)
 		(property "Footprint" ""
-			(at 379.73 43.18 0)
+			(at 363.22 41.91 0)
 			(effects
 				(font
@@
 		)
 		(property "Datasheet" "~"
-			(at 379.73 43.18 0)
+			(at 363.22 41.91 0)
 			(effects
 				(font
@@
 		)
 		(property "Description" "Generic connector, single row, 01x01, script generated"
-			(at 379.73 43.18 0)
+			(at 363.22 41.91 0)
 			(effects
 				(font
@@
 			)
 		)
-		(property "Value" "15"
+		(property "Value" "0.51 Ohms"
 			(at 105.41 241.3 90)
 			(effects
@@
 	(symbol
 		(lib_id "Device:Q_NPN_BCE")
-		(at 349.25 52.07 0)
+		(at 332.74 50.8 0)
 		(unit 1)
 		(exclude_from_sim no)
@@
 		(fields_autoplaced yes)
 		(property "Reference" "Q1"
-			(at 354.33 50.7999 0)
+			(at 337.82 49.5299 0)
 			(effects
 				(font
@@
 		)
 		(property "Value" "KTC4373Y"
-			(at 354.33 53.3399 0)
+			(at 337.82 52.0699 0)
 			(effects
 				(font
@@
 		)
 		(property "Footprint" ""
-			(at 354.33 49.53 0)
+			(at 337.82 48.26 0)
 			(effects
 				(font
@@
 		)
 		(property "Datasheet" "~"
-			(at 349.25 52.07 0)
+			(at 332.74 50.8 0)
 			(effects
 				(font
@@
 		)
 		(property "Description" "NPN transistor, base/collector/emitter"
-			(at 349.25 52.07 0)
+			(at 332.74 50.8 0)
 			(effects
 				(font
@@
 	(symbol
 		(lib_id "power:+BATT")
-		(at 351.79 29.21 0)
+		(at 335.28 27.94 0)
 		(unit 1)
 		(exclude_from_sim no)
@@
 		(fields_autoplaced yes)
 		(property "Reference" "#PWR058"
-			(at 351.79 33.02 0)
+			(at 335.28 31.75 0)
 			(effects
 				(font
@@
 		)
 		(property "Value" "+BATT"
-			(at 351.79 24.13 0)
+			(at 335.28 22.86 0)
 			(effects
 				(font
@@
 		)
 		(property "Footprint" ""
-			(at 351.79 29.21 0)
+			(at 335.28 27.94 0)
 			(effects
 				(font
@@
 		)
 		(property "Datasheet" ""
-			(at 351.79 29.21 0)
+			(at 335.28 27.94 0)
 			(effects
 				(font
@@
 		)
 		(property "Description" "Power symbol creates a global label with name \"+BATT\""
-			(at 351.79 29.21 0)
+			(at 335.28 27.94 0)
 			(effects
 				(font
@@
 	(symbol
 		(lib_id "Connector:Conn_01x01_Pin")
-		(at 379.73 33.02 180)
+		(at 363.22 31.75 180)
 		(unit 1)
 		(exclude_from_sim no)
@@
 		(fields_autoplaced yes)
 		(property "Reference" "T4"
-			(at 379.095 27.94 0)
+			(at 362.585 26.67 0)
 			(effects
 				(font
@@
 		)
 		(property "Value" "SHOCKER_OUTPUT_1"
-			(at 379.095 30.48 0)
+			(at 362.585 29.21 0)
 			(effects
 				(font
@@
 		)
 		(property "Footprint" ""
-			(at 379.73 33.02 0)
+			(at 363.22 31.75 0)
 			(effects
 				(font
@@
 		)
 		(property "Datasheet" "~"
-			(at 379.73 33.02 0)
+			(at 363.22 31.75 0)
 			(effects
 				(font
@@
 		)
 		(property "Description" "Generic connector, single row, 01x01, script generated"
-			(at 379.73 33.02 0)
+			(at 363.22 31.75 0)
 			(effects
 				(font
@@
 	(symbol
 		(lib_id "Device:R_US")
-		(at 336.55 52.07 90)
+		(at 320.04 50.8 90)
 		(unit 1)
 		(exclude_from_sim no)
@@
 		(fields_autoplaced yes)
 		(property "Reference" "R2"
-			(at 336.55 45.72 90)
+			(at 320.04 44.45 90)
 			(effects
 				(font
@@
 			)
 		)
-		(property "Value" "?"
-			(at 336.55 48.26 90)
+		(property "Value" "56 Ohms"
+			(at 320.04 46.99 90)
 			(effects
 				(font
@@
 		)
 		(property "Footprint" ""
-			(at 336.804 51.054 90)
+			(at 320.294 49.784 90)
 			(effects
 				(font
@@
 		)
 		(property "Datasheet" "~"
-			(at 336.55 52.07 0)
+			(at 320.04 50.8 0)
 			(effects
 				(font
@@
 		)
 		(property "Description" "Resistor, US symbol"
-			(at 336.55 52.07 0)
+			(at 320.04 50.8 0)
 			(effects
 				(font
@@
 	(symbol
 		(lib_id "Transformer:TRANSF1")
-		(at 356.87 38.1 0)
+		(at 340.36 36.83 0)
 		(unit 1)
 		(exclude_from_sim no)
@@
 		(dnp no)
 		(property "Reference" "L3"
-			(at 356.87 31.242 0)
+			(at 340.36 29.972 0)
 			(effects
 				(font
@@
 		)
 		(property "Value" "~"
-			(at 356.87 31.75 0)
+			(at 340.36 30.48 0)
 			(effects
 				(font
@@
 		)
 		(property "Footprint" ""
-			(at 356.87 38.1 0)
+			(at 340.36 36.83 0)
 			(effects
 				(font
@@
 		)
 		(property "Datasheet" ""
-			(at 356.87 38.1 0)
+			(at 340.36 36.83 0)
 			(effects
 				(font
@@
 		)
 		(property "Description" ""
-			(at 356.87 38.1 0)
+			(at 340.36 36.83 0)
 			(effects
 				(font
